File: schematics/Pdidi/Схема платы (2).brd (EAGLE design)
At the start: 44 x 35 mm, 29 parts, among them M0 CONNECT_3, M1 CONNECT_3, X1 SD, X2 MK_AB

Commit message: Функция парса
Parts:
- removed AB: (no value), pinhead:1X02
- removed CONCEVIK: (no value), pinhead:1X03
- removed JP1: Klemmnik, pinhead:1X02
- removed JP2: Thermistor, pinhead:1X02
- removed X1: SD, pinhead:1X04
- removed X2: MK_AB, pinhead:1X03
- added 2K: (no value), rcl:R0603
- added AO3407: AO3407, Banka-2026:SOT23-3
- added C3: (no value), rcl:C0603
- added LED1: (no value), led:CHIP-LED0603
- added U$10: SD, UNKNOWN-2024:53047-04
- added U$3: Thermistor, UNKNOWN-2024:53047-02
- added U$9: MK_AB, UNKNOWN-2024:53047-03
- added X3: AB, UNKNOWN-2024:JST-2-2.5
- added X4: Klemmnik, UNKNOWN-2024:JST-2-2.5
- R9: value 10k -> 2k
- U$11: value AO3407 -> CONCEVIK; device Banka-2026:SOT23-3 -> UNKNOWN-2024:53047-03
- moved U$11 18.3 mm to (22.9, 1.80)
Connections:
- new net N$4: 2K.2, LED1.A
- new net N$5: LED1.C, U$5.P$24
- net 3V3: now also AO3407.2, C3.1, U$3.1; no longer JP2.2
- net AB: now also U$9.3; no longer X2.3
- net CS: now also U$10.1; no longer X1.4
- net GND: now also C3.2, U$11.3, U$9.1, U$9.2, X3.1; no longer AB.2, CONCEVIK.1, X2.1, X2.2
- net MISO: now also U$10.4; no longer X1.1
- net MOSI: now also U$10.2; no longer X1.3
- net N$1: now also U$3.2; no longer JP2.1
- net N$11: now also X4.1; no longer JP1.2
- net N$14: now also AO3407.3; no longer U$11.3
- net N$15: now also AO3407.1; no longer CONCEVIK.3
- net N$2: now also U$11.2; no longer CONCEVIK.2
- net SCK: now also U$10.3; no longer X1.2
- net VBAT: now also 2K.1, X3.2, X4.2; no longer AB.1, JP1.1, U$11.2
Routing:
- net N$5: track 0.00 -> 19.1 mm, vias 0 -> 2
- net 3V3: track 82.3 -> 94.3 mm, vias 3 -> 4
- net GND: track 191.8 -> 195.6 mm, vias 7 -> 9
- net AB: track 19.7 -> 22.8 mm
- net SCK: track 9.11 -> 12.2 mm, vias 0 -> 1
- net CS: track 14.9 -> 12.8 mm
- net VBAT: track 107.1 -> 108.9 mm
- net N$4: track 0.00 -> 1.80 mm
- net N$2: track 2.69 -> 3.71 mm
- net MOSI: track 12.2 -> 11.3 mm
- net N$15: track 35.9 -> 35.1 mm
- net MISO: track 5.39 -> 6.12 mm
Other:
- board text added: "100nF"
- board text added: "AO3407"
- board text added: "C"
- board text added: "G"
- board text added: "V"
