File: schematics/Pdidi/Схема платы копия.sch (EAGLE design)
At the start: 29 parts, among them M0 CONNECT_3, M1 CONNECT_3, X1 SD, X2 MK_AB

Commit message: Функция парса
Parts:
- removed AB: (no value), pinhead:PINHD-1X2
- removed CONCEVIK: (no value), pinhead:PINHD-1X3
- removed JP1: Klemmnik, pinhead:PINHD-1X2
- removed JP2: Thermistor, pinhead:PINHD-1X2
- removed X1: SD, pinhead:PINHD-1X4
- removed X2: MK_AB, pinhead:PINHD-1X3
- added 2K: (no value), rcl:R-EU_R0603
- added AO3407: AO3407, Banka-2026:AO3407
- added C3: (no value), rcl:C-EUC0603
- added LED1: (no value), led:LEDCHIP-LED0603
- added U$10: SD, UNKNOWN-2024:MOLEX-4-1.25
- added U$3: Thermistor, UNKNOWN-2024:MOLEX-2-1.25
- added U$9: MK_AB, UNKNOWN-2024:MOLEX-3-1.25
- added X3: AB, UNKNOWN-2024:JST-2-2.5
- added X4: Klemmnik, UNKNOWN-2024:JST-2-2.5
- R9: value 10k -> 2k
- U$11: value AO3407 -> CONCEVIK; device Banka-2026:AO3407 -> UNKNOWN-2024:MOLEX-3-1.25
Connections:
- new net N$4: 2K.2, LED1.A
- new net N$5: LED1.C, U$5.AUX
- net 3V3: now also AO3407.PS, C3.1, U$3.1; no longer JP2.2
- net AB: now also U$9.3; no longer X2.3
- net CS: now also U$10.1; no longer X1.4
- net GND: now also C3.2, U$11.3, U$9.1, U$9.2, X3.1; no longer AB.2, CONCEVIK.1, X2.1, X2.2
- net MISO: now also U$10.4; no longer X1.1
- net MOSI: now also U$10.2; no longer X1.3
- net N$1: now also U$3.2; no longer JP2.1
- net N$11: now also X4.1; no longer JP1.2
- net N$14: now also AO3407.PD; no longer U$11.PD
- net N$15: now also AO3407.PG, U$11.1; no longer CONCEVIK.3, U$11.PG
- net N$2: now also U$11.2; no longer CONCEVIK.2
- net SCK: now also U$10.3; no longer X1.2
- net VBAT: now also 2K.1, X3.2, X4.2; no longer AB.1, JP1.1, U$11.PS
Other:
- moved on the sheet: AMS1117, C1, C2, M0, M1, R1, R2, R4, R5, R6, R7, R8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
